File: PC-AXE.kicad_pcb (KiCad board)
At the start: 4 copper layers, 312 x 111.2 mm, 563 parts, among them J1 PCIexpress_bracket, J10 61900411021, J2 PCIexpress_x4, J3 353180620, J4 353180620, J5 353180620, J6 Conn_01x06, J7 61900411021, J8 61900411021, J9 61900411021, U1 TLV62568ADRLR, U10 CSD95472Q5MC, U11 CSD95472Q5MC, U12 CSD95472Q5MC, U13 25MHz, U14 TXU0304PW, U15 MCP1824T-0802E, U16 MCP1824T-1202E, U17 BM1370_mode1, U18 BM1370_mode1, U19 BM1370_mode1, U2 AP2204K-1.8, U20 BM1370_mode1, U21 BM1370_mode1, U22 BM1370_mode1, U23 BM1370_mode1, U24 BM1370_mode1, U25 BM1370_mode1, U26 BM1370_mode1, U27 BM1370_mode1, U28 BM1370_mode1, U29 EMC2305, U3 VL805, U30 M93C46-WDW6TP, U31 FT4232HQ, U4 W25Q32JVZP, U5 AP3211, U6 TPS53667RTAR, U7 CSD95472Q5MC, U8 CSD95472Q5MC, U9 CSD95472Q5MC, Y1 25Mhz, Y2 12MHz

Commit message: board stakup updated and schematic is updated
Parts:
- removed C1: 10uF, Capacitor_SMD:C_0603_1608Metric
- removed C10, C11, C12, C13, C14, C16, C17, C18, C19, C23, C24, C27, C3, C4, C5, C6, C7, C8, C9: 100nF, Capacitor_SMD:C_0402_1005Metric
- removed C100, C101, C102, C103, C104, C105, C106, C107, C108, C59, C62, C65, C66, C69, C72, C73, C76, C77, C80, C81, C84, C85, C88, C89, C92, C93, C96, C97, C98, C99: 330µF/4V, Capacitor_SMD:C_1210_3225Metric
- removed C109, C117, C127, C137, C147, C157, C38, C39, C41, C42, C43, C44, C45, C46, C47, C48, C49, C50, C53: 22µ/25V, Capacitor_SMD:C_1210_3225Metric
- removed C110, C118, C128, C138, C148, C158, C169, C171, C180, C196, C212, C228, C244, C260, C276, C292, C308, C324, C340, C356, C52, C54: 1µF/25V, Capacitor_SMD:C_0805_2012Metric
- removed C111, C116, C119, C124, C129, C134, C139, C144, C149, C154, C159, C164, C36, C37, C58: 1nF, Capacitor_SMD:C_0805_2012Metric
- removed C112, C113, C115, C120, C121, C123, C130, C131, C133, C140, C141, C143, C150, C151, C153, C160, C161, C163, C165, C166, C167, C168, C170, C182, C198, C214, C230, C246, C262, C278, C294, C310, C326, C342, C358: 100nF, Capacitor_SMD:C_0805_2012Metric
- removed C114, C122, C132, C142, C152, C162: 2.2µF/16V, Capacitor_SMD:C_0805_2012Metric
- removed C15, C2: 10uF, Capacitor_SMD:C_0402_1005Metric
- removed C172, C173, C174, C175, C176, C178, C181, C183, C184, C185, C186, C187, C188, C189, C190, C191, C192, C194, C197, C199, C200, C201, C202, C203, C204, C205, C206, C207, C208, C210, C213, C215, C216, C217, C218, C219, C220, C221, C222, C223, C224, C226, C229, C231, C232, C233, C234, C235, C236, C237, C238, C239, C240, C242, C245, C247, C248, C249, C250, C251, C252, C253, C254, C255, C256, C258, C261, C263, C264, C265, C266, C267, C268, C269, C270, C271, C272, C274, C277, C279, C280, C281, C282, C283, C284, C285, C286, C287, C288, C290, C293, C295, C296, C297, C298, C299, C300, C301, C302, C303, C304, C306, C309, C311, C312, C313, C314, C315, C316, C317, C318, C319, C320, C322, C325, C327, C328, C329, C330, C331, C332, C333, C334, C335, C336, C338, C341, C343, C344, C345, C346, C347, C348, C349, C350, C351, C352, C354, C357, C359, C360, C361, C362, C363: 1µF/6.3V, Capacitor_SMD:C_0603_1608Metric_Pad1.08x0.95mm_HandSolder
- removed C177, C193, C209, C225, C241, C257, C273, C289, C305, C31, C321, C337, C353: 10µF/25V, Capacitor_SMD:C_0805_2012Metric
- removed C179, C195, C211, C227, C243, C259, C275, C291, C307, C323, C339, C355, C60, C61, C63, C64, C67, C68, C70, C71, C74, C75, C78, C79, C82, C83, C86, C87, C90, C91, C94, C95: 100µ/6.3V, Capacitor_SMD:C_1206_3216Metric
- removed C20: 10pF, Capacitor_SMD:C_0402_1005Metric
- removed C21: 1uF, Capacitor_SMD:C_0402_1005Metric
- removed C22: 22uF, Capacitor_SMD:C_0603_1608Metric
- removed C25, C26: 18pF, Capacitor_SMD:C_0402_1005Metric
- removed C28, C29, C30, C32: 470µ/25V, Capacitor_SMD:CP_Elec_8x10
- removed C33, C35: 22pF, Capacitor_SMD:C_0805_2012Metric
- removed C34: 100pF, Capacitor_SMD:C_0805_2012Metric
- removed C364, C369, C371, C372, C373, C374, C375, C376, C377, C378: 0.1uF, Capacitor_SMD:C_0805_2012Metric
- removed C365, C368: 27pf, Capacitor_SMD:C_0805_2012Metric
- removed C366, C367: 4.7uF, Capacitor_SMD:C_0805_2012Metric
- removed C370: 3.3uF, Capacitor_SMD:C_0805_2012Metric
- removed C40: 10nF, Capacitor_SMD:C_0805_2012Metric
- removed C51: 4.7µF/16V, Capacitor_SMD:C_0805_2012Metric
- removed C55: 330nF, Capacitor_SMD:C_0805_2012Metric
- removed C56: 12pF, Capacitor_SMD:C_0805_2012Metric
- removed C57: 2.2nF, Capacitor_SMD:C_0805_2012Metric
- removed D1: PMEG4030EP,115, Diode_SMD:D_SOD-128
- removed FB1, FB2: FerriteBead_Small, Resistor_SMD:R_0603_1608Metric
- removed J10, J7, J8, J9: 61900411021, bitcrane:CONN-TH_4P-P2.54_HCTL_HC-2510-4AW
- removed J3, J4, J5: 353180620, 353180620:MOLEX_353180620
- removed J6: Conn_01x06, Connector_PinHeader_1.27mm:PinHeader_1x06_P1.27mm_Vertical
- removed L1: 1uH, Inductor_SMD:L_Vishay_IHLP-1212
- removed L2: 4.7µH, Inductor_SMD:L_Taiyo-Yuden_NR-50xx
- removed L3, L4, L5, L6, L7, L8: 220nH, IFLR-4031GC-01-8x10:IFLR-4031GC-01-8x10
- removed NT1, NT2: NetTie_2, NetTie:NetTie-2_SMD_Pad0.5mm
- removed R10: 6.04K, Resistor_SMD:R_0402_1005Metric
- removed R100, R91, R92, R93, R94, R95, R98: 10k, Resistor_SMD:R_0805_2012Metric
- removed R101: 12k, Resistor_SMD:R_0805_2012Metric
- removed R102: 1k, Resistor_SMD:R_0805_2012Metric
- removed R11: 15K, Resistor_SMD:R_0402_1005Metric
- removed R12, R5, R6: 10K, Resistor_SMD:R_0402_1005Metric
- removed R15, R23: 16.5K, Resistor_SMD:R_0805_2012Metric
- removed R16: 24.3K, Resistor_SMD:R_0805_2012Metric
- removed R17, R18: 51 0.5%, Resistor_SMD:R_0805_2012Metric
- removed R19: 121K, Resistor_SMD:R_0805_2012Metric
- removed R20, R21, R46, R47, R48: 10K, Resistor_SMD:R_0805_2012Metric
- removed R22: 86.6K, Resistor_SMD:R_0805_2012Metric
- removed R24: 2.55K, Resistor_SMD:R_0805_2012Metric
- removed R25: 8.06K, Resistor_SMD:R_0805_2012Metric
- removed R26: 49.9K, Resistor_SMD:R_0805_2012Metric
- removed R27: 100K, Resistor_SMD:R_0805_2012Metric
- removed R28, R29: 2.2R, Resistor_SMD:R_0805_2012Metric
- removed R3: 75K, Resistor_SMD:R_0402_1005Metric
- removed R32, R33, R36, R37, R38, R39, R40, R41, R42, R43, R44, R45: 1R, Resistor_SMD:R_0805_2012Metric
- removed R4: 100K, Resistor_SMD:R_0402_1005Metric
- removed R49, R50, R51, R52, R53, R54, R55, R56, R57, R58, R59: 33R, Resistor_SMD:R_0402_1005Metric_Pad0.72x0.64mm_HandSolder
- removed R60, R62, R64, R66, R68, R70, R72, R74, R76, R78, R80, R82: 1K, Resistor_SMD:R_0805_2012Metric
- removed R61, R63, R65, R67, R69, R71, R73, R75, R77, R79, R81, R83: 2K, Resistor_SMD:R_0805_2012Metric
- removed R7: DNP, Resistor_SMD:R_0402_1005Metric
- removed R84, R97, R99: 4.7k, Resistor_SMD:R_0805_2012Metric
- removed R85: 33k, Resistor_SMD:R_0805_2012Metric
- removed R86: 22k, Resistor_SMD:R_0805_2012Metric
- removed R87, R88, R89, R90: 36k, Resistor_SMD:R_0805_2012Metric
- removed R9: 4.7K, Resistor_SMD:R_0402_1005Metric
- removed R96: 2.2k, Resistor_SMD:R_0805_2012Metric
- removed TP1, TP10, TP11, TP12, TP13, TP14, TP15, TP16, TP2, TP3, TP4, TP5, TP6, TP7, TP8, TP9: TestPoint, TestPoint:TestPoint_Pad_D1.0mm
- removed TP17, TP18, TP19, TP20, TP21, TP22, TP23, TP24, TP25, TP26, TP27: TestPoint, TestPoint:TestPoint_Pad_D1.5mm
- removed U1: TLV62568ADRLR, Package_TO_SOT_SMD:SOT-563
- removed U10, U11, U12, U7, U8, U9: CSD95472Q5MC, CSD95472Q5MC:IC_CSD95490Q5MC
- removed U13: 25MHz, Oscillator:Oscillator_SMD_EuroQuartz_XO32-4Pin_3.2x2.5mm
- removed U14: TXU0304PW, Package_SO:TSSOP-14-1EP_4.4x5mm_P0.65mm
- removed U15: MCP1824T-0802E, Package_TO_SOT_SMD:SOT-23-5
- removed U16: MCP1824T-1202E, Package_TO_SOT_SMD:SOT-23-5
- removed U17, U18, U19, U20, U21, U22, U23, U24, U25, U26, U27, U28: BM1370_mode1, BM1370:BM1370
- removed U2: AP2204K-1.8, Package_TO_SOT_SMD:SOT-23-5
- removed U29: EMC2305, bitcart:QFN16_4x4MC_MCH
- removed U3: VL805, Package_DFN_QFN:QFN-68-1EP_8x8mm_P0.4mm_EP5.2x5.2mm
- removed U30: M93C46-WDW6TP, bitcrane:TSSOP-8_L4.4-W3.0-P0.65-LS6.4-BL
- removed U31: FT4232HQ, bitcrane:QFN50P900X900X105-65N
- removed U4: W25Q32JVZP, Package_DFN_QFN:DFN-8-1EP_3x2mm_P0.5mm_EP1.36x1.46mm
- removed U5: AP3211, Package_TO_SOT_SMD:SOT-23-6
- removed U6: TPS53667RTAR, TPS53667RTAR:IC_TPS53667RTAR
- removed Y1: 25Mhz, Crystal:Crystal_SMD_3225-4Pin_3.2x2.5mm
- removed Y2: 12MHz, Crystal:Crystal_SMD_3225-4Pin_3.2x2.5mm
- moved C135 0.05 mm to (131.9, 183.1), turned to -90 degrees
- turned C155 to -90 degrees
Routing:
- net /PET0_N: track 8.95 -> 10.4 mm
- net /PET2_N: track 8.95 -> 10.4 mm
- net /PCIexpress_connector/_PER1_N: track 5.70 -> 7.10 mm, vias 1 -> 0
- net /PET0_P: track 8.97 -> 10.4 mm
- net /PET3_N: track 5.70 -> 7.09 mm
- net /PET3_P: track 5.70 -> 7.08 mm
- net /PET1_P: track 5.70 -> 7.08 mm
- net /PET1_N: track 5.70 -> 7.08 mm
- net /PCIexpress_connector/_PER2_P: track 5.70 -> 7.08 mm
- net /PCIexpress_connector/_PER2_N: track 5.70 -> 7.08 mm
- net /PET2_P: track 8.97 -> 10.3 mm
- net /PCIexpress_connector/_PER3_P: track 5.70 -> 7.08 mm
- net /PCIexpress_connector/_PER0_P: track 5.70 -> 7.08 mm
- net /PCIexpress_connector/_PER3_N: track 5.70 -> 7.07 mm
- net /PCIexpress_connector/_PER0_N: track 5.70 -> 7.06 mm
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Other:
- copper layers 4 -> 6
- rule pad_to_mask_clearance: 0.051 -> 0

Commit message: updated schematic working on layout
Parts:
- added C1: 10uF, Capacitor_SMD:C_0603_1608Metric, F.Cu at (551.7, 326.1)
- added C10: 100nF, Capacitor_SMD:C_0402_1005Metric, F.Cu at (565.7, 390.3)
- added C100: 330µF/4V, Capacitor_SMD:C_1210_3225Metric, F.Cu at (1010.8, 472.8)
- added C101: 330µF/4V, Capacitor_SMD:C_1210_3225Metric, F.Cu at (1013.3, 472.8)
- added C102: 330µF/4V, Capacitor_SMD:C_1210_3225Metric, F.Cu at (1015.9, 472.8)
- added C103: 330µF/4V, Capacitor_SMD:C_1210_3225Metric, F.Cu at (1018.4, 472.8)
- added C104: 330µF/4V, Capacitor_SMD:C_1210_3225Metric, F.Cu at (1020.9, 472.8)
- added C105: 330µF/4V, Capacitor_SMD:C_1210_3225Metric, F.Cu at (1023.5, 472.8)
- added C106: 330µF/4V, Capacitor_SMD:C_1210_3225Metric, F.Cu at (1026.0, 472.8)
- added C107: 330µF/4V, Capacitor_SMD:C_1210_3225Metric, F.Cu at (1028.6, 472.8)
- added C108: 330µF/4V, Capacitor_SMD:C_1210_3225Metric, F.Cu at (1031.1, 472.8)
- added C109: 22µ/25V, Capacitor_SMD:C_1210_3225Metric, F.Cu at (754.8, 648.1)
- added C11: 100nF, Capacitor_SMD:C_0402_1005Metric, F.Cu at (568.2, 373.8)
- added C110: 1µF/25V, Capacitor_SMD:C_0805_2012Metric, F.Cu at (759.3, 648.1)
- added C111: 1nF, Capacitor_SMD:C_0805_2012Metric, F.Cu at (763.1, 636.6)
- added C112: 100nF, Capacitor_SMD:C_0805_2012Metric, F.Cu at (763.7, 648.1)
- added C113: 100nF, Capacitor_SMD:C_0805_2012Metric, F.Cu at (767.5, 672.8)
- added C114: 2.2µF/16V, Capacitor_SMD:C_0805_2012Metric, F.Cu at (776.4, 672.8)
- added C115: 100nF, Capacitor_SMD:C_0805_2012Metric, F.Cu at (792.3, 658.9)
- added C116: 1nF, Capacitor_SMD:C_0805_2012Metric, F.Cu at (799.9, 673.5)
- added C117: 22µ/25V, Capacitor_SMD:C_1210_3225Metric, F.Cu at (843.5, 649.2)
- added C118: 1µF/25V, Capacitor_SMD:C_0805_2012Metric, F.Cu at (847.9, 649.2)
- added C119: 1nF, Capacitor_SMD:C_0805_2012Metric, F.Cu at (851.7, 637.8)
- added C12: 100nF, Capacitor_SMD:C_0402_1005Metric, F.Cu at (568.2, 390.3)
- added C120: 100nF, Capacitor_SMD:C_0805_2012Metric, F.Cu at (852.4, 649.2)
- added C121: 100nF, Capacitor_SMD:C_0805_2012Metric, F.Cu at (856.2, 674.0)
- added C122: 2.2µF/16V, Capacitor_SMD:C_0805_2012Metric, F.Cu at (865.1, 674.0)
- added C123: 100nF, Capacitor_SMD:C_0805_2012Metric, F.Cu at (880.9, 660.0)
- added C124: 1nF, Capacitor_SMD:C_0805_2012Metric, F.Cu at (888.6, 674.6)
- added C127: 22µ/25V, Capacitor_SMD:C_1210_3225Metric, F.Cu at (657.9, 653.7)
- added C128: 1µF/25V, Capacitor_SMD:C_0805_2012Metric, F.Cu at (662.3, 653.7)
- added C129: 1nF, Capacitor_SMD:C_0805_2012Metric, F.Cu at (666.2, 642.2)
- added C13: 100nF, Capacitor_SMD:C_0402_1005Metric, F.Cu at (570.8, 373.8)
- added C130: 100nF, Capacitor_SMD:C_0805_2012Metric, F.Cu at (666.8, 653.7)
- added C131: 100nF, Capacitor_SMD:C_0805_2012Metric, F.Cu at (670.6, 678.4)
- added C132: 2.2µF/16V, Capacitor_SMD:C_0805_2012Metric, F.Cu at (679.5, 678.4)
- added C133: 100nF, Capacitor_SMD:C_0805_2012Metric, F.Cu at (695.4, 664.5)
- added C134: 1nF, Capacitor_SMD:C_0805_2012Metric, F.Cu at (703.0, 679.1)
- added C137: 22µ/25V, Capacitor_SMD:C_1210_3225Metric, F.Cu at (937.8, 642.7)
- added C138: 1µF/25V, Capacitor_SMD:C_0805_2012Metric, F.Cu at (942.3, 642.7)
- added C139: 1nF, Capacitor_SMD:C_0805_2012Metric, F.Cu at (946.1, 631.2)
- added C14: 100nF, Capacitor_SMD:C_0402_1005Metric, F.Cu at (570.8, 390.3)
- added C140: 100nF, Capacitor_SMD:C_0805_2012Metric, F.Cu at (946.7, 642.7)
- added C141: 100nF, Capacitor_SMD:C_0805_2012Metric, F.Cu at (950.5, 667.4)
- added C142: 2.2µF/16V, Capacitor_SMD:C_0805_2012Metric, F.Cu at (959.4, 667.4)
- added C143: 100nF, Capacitor_SMD:C_0805_2012Metric, F.Cu at (975.3, 653.5)
- added C144: 1nF, Capacitor_SMD:C_0805_2012Metric, F.Cu at (982.9, 668.1)
- added C147: 22µ/25V, Capacitor_SMD:C_1210_3225Metric, F.Cu at (1028.7, 642.6)
- added C148: 1µF/25V, Capacitor_SMD:C_0805_2012Metric, F.Cu at (1033.2, 642.6)
- added C149: 1nF, Capacitor_SMD:C_0805_2012Metric, F.Cu at (1037.0, 631.2)
- added C15: 10uF, Capacitor_SMD:C_0402_1005Metric, F.Cu at (572.0, 346.5)
- added C150: 100nF, Capacitor_SMD:C_0805_2012Metric, F.Cu at (1037.6, 642.6)
- added C151: 100nF, Capacitor_SMD:C_0805_2012Metric, F.Cu at (1041.4, 667.4)
- added C152: 2.2µF/16V, Capacitor_SMD:C_0805_2012Metric, F.Cu at (1050.3, 667.4)
- added C153: 100nF, Capacitor_SMD:C_0805_2012Metric, F.Cu at (1066.2, 653.4)
- added C154: 1nF, Capacitor_SMD:C_0805_2012Metric, F.Cu at (1073.8, 668.0)
- added C157: 22µ/25V, Capacitor_SMD:C_1210_3225Metric, F.Cu at (1139.1, 647.3)
- added C158: 1µF/25V, Capacitor_SMD:C_0805_2012Metric, F.Cu at (1143.5, 647.3)
- added C159: 1nF, Capacitor_SMD:C_0805_2012Metric, F.Cu at (1147.3, 635.9)
- added C16: 100nF, Capacitor_SMD:C_0402_1005Metric, F.Cu at (573.3, 373.8)
- added C160: 100nF, Capacitor_SMD:C_0805_2012Metric, F.Cu at (1148.0, 647.3)
- added C161: 100nF, Capacitor_SMD:C_0805_2012Metric, F.Cu at (1151.8, 672.1)
- added C162: 2.2µF/16V, Capacitor_SMD:C_0805_2012Metric, F.Cu at (1160.7, 672.1)
- added C163: 100nF, Capacitor_SMD:C_0805_2012Metric, F.Cu at (1176.5, 658.1)
- added C164: 1nF, Capacitor_SMD:C_0805_2012Metric, F.Cu at (1184.2, 672.7)
- added C165: 100nF, Capacitor_SMD:C_0805_2012Metric, F.Cu at (818.1, 125.1)
- added C166: 100nF, Capacitor_SMD:C_0805_2012Metric, F.Cu at (827.6, 93.1)
- added C167: 100nF, Capacitor_SMD:C_0805_2012Metric, F.Cu at (830.8, 167.7)
- added C168: 100nF, Capacitor_SMD:C_0805_2012Metric, F.Cu at (845.4, 92.4)
- added C169: 1µF/25V, Capacitor_SMD:C_0805_2012Metric, F.Cu at (848.6, 168.3)
- added C17: 100nF, Capacitor_SMD:C_0402_1005Metric, F.Cu at (573.3, 390.3)
- added C170: 100nF, Capacitor_SMD:C_0805_2012Metric, F.Cu at (859.4, 167.7)
- added C171: 1µF/25V, Capacitor_SMD:C_0805_2012Metric, F.Cu at (877.8, 168.3)
- added C172: 1µF/6.3V, Capacitor_SMD:C_0603_1608Metric_Pad1.08x0.95mm_HandSolder, F.Cu at (644.3, 823.0)
- added C173: 1µF/6.3V, Capacitor_SMD:C_0603_1608Metric_Pad1.08x0.95mm_HandSolder, F.Cu at (648.1, 823.0)
- added C174: 1µF/6.3V, Capacitor_SMD:C_0603_1608Metric_Pad1.08x0.95mm_HandSolder, F.Cu at (648.7, 791.3)
- added C175: 1µF/6.3V, Capacitor_SMD:C_0603_1608Metric_Pad1.08x0.95mm_HandSolder, F.Cu at (654.4, 791.3)
- added C176: 1µF/6.3V, Capacitor_SMD:C_0603_1608Metric_Pad1.08x0.95mm_HandSolder, F.Cu at (660.1, 791.3)
- added C177: 10µF/25V, Capacitor_SMD:C_0805_2012Metric, F.Cu at (664.6, 828.1)
- added C178: 1µF/6.3V, Capacitor_SMD:C_0603_1608Metric_Pad1.08x0.95mm_HandSolder, F.Cu at (668.4, 791.3)
- added C179: 100µ/6.3V, Capacitor_SMD:C_1206_3216Metric, F.Cu at (672.8, 777.9)
- added C18: 100nF, Capacitor_SMD:C_0402_1005Metric, F.Cu at (575.8, 373.8)
- added C180: 1µF/25V, Capacitor_SMD:C_0805_2012Metric, F.Cu at (672.8, 828.1)
- added C181: 1µF/6.3V, Capacitor_SMD:C_0603_1608Metric_Pad1.08x0.95mm_HandSolder, F.Cu at (678.5, 791.3)
- added C182: 100nF, Capacitor_SMD:C_0805_2012Metric, F.Cu at (681.7, 828.1)
- added C183: 1µF/6.3V, Capacitor_SMD:C_0603_1608Metric_Pad1.08x0.95mm_HandSolder, F.Cu at (685.5, 791.3)
- added C184: 1µF/6.3V, Capacitor_SMD:C_0603_1608Metric_Pad1.08x0.95mm_HandSolder, F.Cu at (691.9, 791.3)
- added C185: 1µF/6.3V, Capacitor_SMD:C_0603_1608Metric_Pad1.08x0.95mm_HandSolder, F.Cu at (693.8, 823.0)
- added C186: 1µF/6.3V, Capacitor_SMD:C_0603_1608Metric_Pad1.08x0.95mm_HandSolder, F.Cu at (697.0, 823.0)
- added C187: 1µF/6.3V, Capacitor_SMD:C_0603_1608Metric_Pad1.08x0.95mm_HandSolder, F.Cu at (697.6, 791.3)
- added C188: 1µF/6.3V, Capacitor_SMD:C_0603_1608Metric_Pad1.08x0.95mm_HandSolder, F.Cu at (742.9, 820.3)
- added C189: 1µF/6.3V, Capacitor_SMD:C_0603_1608Metric_Pad1.08x0.95mm_HandSolder, F.Cu at (746.7, 820.3)
- added C19: 100nF, Capacitor_SMD:C_0402_1005Metric, F.Cu at (575.8, 390.3)
- added C190: 1µF/6.3V, Capacitor_SMD:C_0603_1608Metric_Pad1.08x0.95mm_HandSolder, F.Cu at (747.3, 788.6)
- added C191: 1µF/6.3V, Capacitor_SMD:C_0603_1608Metric_Pad1.08x0.95mm_HandSolder, F.Cu at (753.0, 788.6)
- added C192: 1µF/6.3V, Capacitor_SMD:C_0603_1608Metric_Pad1.08x0.95mm_HandSolder, F.Cu at (758.7, 788.6)
- added C193: 10µF/25V, Capacitor_SMD:C_0805_2012Metric, F.Cu at (763.2, 825.4)
- added C194: 1µF/6.3V, Capacitor_SMD:C_0603_1608Metric_Pad1.08x0.95mm_HandSolder, F.Cu at (767.0, 788.6)
- added C195: 100µ/6.3V, Capacitor_SMD:C_1206_3216Metric, F.Cu at (771.4, 775.2)
- added C196: 1µF/25V, Capacitor_SMD:C_0805_2012Metric, F.Cu at (771.4, 825.4)
- added C197: 1µF/6.3V, Capacitor_SMD:C_0603_1608Metric_Pad1.08x0.95mm_HandSolder, F.Cu at (777.1, 788.6)
- added C198: 100nF, Capacitor_SMD:C_0805_2012Metric, F.Cu at (780.3, 825.4)
- added C199: 1µF/6.3V, Capacitor_SMD:C_0603_1608Metric_Pad1.08x0.95mm_HandSolder, F.Cu at (784.1, 788.6)
- added C2: 10uF, Capacitor_SMD:C_0402_1005Metric, F.Cu at (556.8, 346.5)
- added C20: 10pF, Capacitor_SMD:C_0402_1005Metric, F.Cu at (579.6, 326.1)
- added C200: 1µF/6.3V, Capacitor_SMD:C_0603_1608Metric_Pad1.08x0.95mm_HandSolder, F.Cu at (790.5, 788.6)
- added C201: 1µF/6.3V, Capacitor_SMD:C_0603_1608Metric_Pad1.08x0.95mm_HandSolder, F.Cu at (792.4, 820.3)
- added C202: 1µF/6.3V, Capacitor_SMD:C_0603_1608Metric_Pad1.08x0.95mm_HandSolder, F.Cu at (795.6, 820.3)
- added C203: 1µF/6.3V, Capacitor_SMD:C_0603_1608Metric_Pad1.08x0.95mm_HandSolder, F.Cu at (796.2, 788.6)
- added C204: 1µF/6.3V, Capacitor_SMD:C_0603_1608Metric_Pad1.08x0.95mm_HandSolder, F.Cu at (840.4, 829.3)
- added C205: 1µF/6.3V, Capacitor_SMD:C_0603_1608Metric_Pad1.08x0.95mm_HandSolder, F.Cu at (844.2, 829.3)
- added C206: 1µF/6.3V, Capacitor_SMD:C_0603_1608Metric_Pad1.08x0.95mm_HandSolder, F.Cu at (844.8, 797.6)
- added C207: 1µF/6.3V, Capacitor_SMD:C_0603_1608Metric_Pad1.08x0.95mm_HandSolder, F.Cu at (850.5, 797.6)
- added C208: 1µF/6.3V, Capacitor_SMD:C_0603_1608Metric_Pad1.08x0.95mm_HandSolder, F.Cu at (856.2, 797.6)
- added C209: 10µF/25V, Capacitor_SMD:C_0805_2012Metric, F.Cu at (860.7, 834.4)
- added C21: 1uF, Capacitor_SMD:C_0402_1005Metric, F.Cu at (585.4, 352.2)
- added C210: 1µF/6.3V, Capacitor_SMD:C_0603_1608Metric_Pad1.08x0.95mm_HandSolder, F.Cu at (864.5, 797.6)
- added C211: 100µ/6.3V, Capacitor_SMD:C_1206_3216Metric, F.Cu at (868.9, 784.2)
- added C212: 1µF/25V, Capacitor_SMD:C_0805_2012Metric, F.Cu at (868.9, 834.4)
- added C213: 1µF/6.3V, Capacitor_SMD:C_0603_1608Metric_Pad1.08x0.95mm_HandSolder, F.Cu at (874.7, 797.6)
- added C214: 100nF, Capacitor_SMD:C_0805_2012Metric, F.Cu at (877.8, 834.4)
- added C215: 1µF/6.3V, Capacitor_SMD:C_0603_1608Metric_Pad1.08x0.95mm_HandSolder, F.Cu at (881.6, 797.6)
- added C216: 1µF/6.3V, Capacitor_SMD:C_0603_1608Metric_Pad1.08x0.95mm_HandSolder, F.Cu at (888.0, 797.6)
- added C217: 1µF/6.3V, Capacitor_SMD:C_0603_1608Metric_Pad1.08x0.95mm_HandSolder, F.Cu at (889.9, 829.3)
- added C218: 1µF/6.3V, Capacitor_SMD:C_0603_1608Metric_Pad1.08x0.95mm_HandSolder, F.Cu at (893.1, 829.3)
- added C219: 1µF/6.3V, Capacitor_SMD:C_0603_1608Metric_Pad1.08x0.95mm_HandSolder, F.Cu at (893.7, 797.6)
- added C22: 22uF, Capacitor_SMD:C_0603_1608Metric, F.Cu at (586.0, 326.1)
- added C220: 1µF/6.3V, Capacitor_SMD:C_0603_1608Metric_Pad1.08x0.95mm_HandSolder, F.Cu at (932.2, 831.0)
- added C221: 1µF/6.3V, Capacitor_SMD:C_0603_1608Metric_Pad1.08x0.95mm_HandSolder, F.Cu at (936.0, 831.0)
- added C222: 1µF/6.3V, Capacitor_SMD:C_0603_1608Metric_Pad1.08x0.95mm_HandSolder, F.Cu at (936.6, 799.3)
- added C223: 1µF/6.3V, Capacitor_SMD:C_0603_1608Metric_Pad1.08x0.95mm_HandSolder, F.Cu at (942.3, 799.3)
- added C224: 1µF/6.3V, Capacitor_SMD:C_0603_1608Metric_Pad1.08x0.95mm_HandSolder, F.Cu at (948.0, 799.3)
- added C225: 10µF/25V, Capacitor_SMD:C_0805_2012Metric, F.Cu at (952.5, 836.1)
- added C226: 1µF/6.3V, Capacitor_SMD:C_0603_1608Metric_Pad1.08x0.95mm_HandSolder, F.Cu at (956.3, 799.3)
- added C227: 100µ/6.3V, Capacitor_SMD:C_1206_3216Metric, F.Cu at (960.7, 786.0)
- added C228: 1µF/25V, Capacitor_SMD:C_0805_2012Metric, F.Cu at (960.7, 836.1)
- added C229: 1µF/6.3V, Capacitor_SMD:C_0603_1608Metric_Pad1.08x0.95mm_HandSolder, F.Cu at (966.5, 799.3)
- added C23: 100nF, Capacitor_SMD:C_0402_1005Metric, F.Cu at (599.3, 340.8)
- added C230: 100nF, Capacitor_SMD:C_0805_2012Metric, F.Cu at (969.6, 836.1)
- added C231: 1µF/6.3V, Capacitor_SMD:C_0603_1608Metric_Pad1.08x0.95mm_HandSolder, F.Cu at (973.4, 799.3)
- added C232: 1µF/6.3V, Capacitor_SMD:C_0603_1608Metric_Pad1.08x0.95mm_HandSolder, F.Cu at (979.8, 799.3)
- added C233: 1µF/6.3V, Capacitor_SMD:C_0603_1608Metric_Pad1.08x0.95mm_HandSolder, F.Cu at (981.7, 831.0)
- added C234: 1µF/6.3V, Capacitor_SMD:C_0603_1608Metric_Pad1.08x0.95mm_HandSolder, F.Cu at (984.9, 831.0)
- added C235: 1µF/6.3V, Capacitor_SMD:C_0603_1608Metric_Pad1.08x0.95mm_HandSolder, F.Cu at (985.5, 799.3)
- added C236: 1µF/6.3V, Capacitor_SMD:C_0603_1608Metric_Pad1.08x0.95mm_HandSolder, F.Cu at (1032.8, 831.0)
- added C237: 1µF/6.3V, Capacitor_SMD:C_0603_1608Metric_Pad1.08x0.95mm_HandSolder, F.Cu at (1036.6, 831.0)
- added C238: 1µF/6.3V, Capacitor_SMD:C_0603_1608Metric_Pad1.08x0.95mm_HandSolder, F.Cu at (1037.2, 799.2)
- added C239: 1µF/6.3V, Capacitor_SMD:C_0603_1608Metric_Pad1.08x0.95mm_HandSolder, F.Cu at (1042.9, 799.2)
- added C24: 100nF, Capacitor_SMD:C_0402_1005Metric, F.Cu at (599.3, 342.0)
- added C240: 1µF/6.3V, Capacitor_SMD:C_0603_1608Metric_Pad1.08x0.95mm_HandSolder, F.Cu at (1048.6, 799.2)
- added C241: 10µF/25V, Capacitor_SMD:C_0805_2012Metric, F.Cu at (1053.1, 836.1)
- added C242: 1µF/6.3V, Capacitor_SMD:C_0603_1608Metric_Pad1.08x0.95mm_HandSolder, F.Cu at (1056.9, 799.2)
- added C243: 100µ/6.3V, Capacitor_SMD:C_1206_3216Metric, F.Cu at (1061.3, 785.9)
- added C244: 1µF/25V, Capacitor_SMD:C_0805_2012Metric, F.Cu at (1061.3, 836.1)
- added C245: 1µF/6.3V, Capacitor_SMD:C_0603_1608Metric_Pad1.08x0.95mm_HandSolder, F.Cu at (1067.0, 799.2)
- added C246: 100nF, Capacitor_SMD:C_0805_2012Metric, F.Cu at (1070.2, 836.1)
- added C247: 1µF/6.3V, Capacitor_SMD:C_0603_1608Metric_Pad1.08x0.95mm_HandSolder, F.Cu at (1074.0, 799.2)
- added C248: 1µF/6.3V, Capacitor_SMD:C_0603_1608Metric_Pad1.08x0.95mm_HandSolder, F.Cu at (1080.4, 799.2)
- added C249: 1µF/6.3V, Capacitor_SMD:C_0603_1608Metric_Pad1.08x0.95mm_HandSolder, F.Cu at (1082.3, 831.0)
- added C25: 18pF, Capacitor_SMD:C_0402_1005Metric, F.Cu at (630.4, 383.9)
- added C250: 1µF/6.3V, Capacitor_SMD:C_0603_1608Metric_Pad1.08x0.95mm_HandSolder, F.Cu at (1085.5, 831.0)
- added C251: 1µF/6.3V, Capacitor_SMD:C_0603_1608Metric_Pad1.08x0.95mm_HandSolder, F.Cu at (1086.1, 799.2)
- added C252: 1µF/6.3V, Capacitor_SMD:C_0603_1608Metric_Pad1.08x0.95mm_HandSolder, F.Cu at (1132.3, 827.9)
- added C253: 1µF/6.3V, Capacitor_SMD:C_0603_1608Metric_Pad1.08x0.95mm_HandSolder, F.Cu at (1136.1, 827.9)
- added C254: 1µF/6.3V, Capacitor_SMD:C_0603_1608Metric_Pad1.08x0.95mm_HandSolder, F.Cu at (1136.7, 796.2)
- added C255: 1µF/6.3V, Capacitor_SMD:C_0603_1608Metric_Pad1.08x0.95mm_HandSolder, F.Cu at (1142.4, 796.2)
- added C256: 1µF/6.3V, Capacitor_SMD:C_0603_1608Metric_Pad1.08x0.95mm_HandSolder, F.Cu at (1148.1, 796.2)
- added C257: 10µF/25V, Capacitor_SMD:C_0805_2012Metric, F.Cu at (1152.6, 833.0)
- added C258: 1µF/6.3V, Capacitor_SMD:C_0603_1608Metric_Pad1.08x0.95mm_HandSolder, F.Cu at (1156.4, 796.2)
- added C259: 100µ/6.3V, Capacitor_SMD:C_1206_3216Metric, F.Cu at (1160.8, 782.9)
- added C26: 18pF, Capacitor_SMD:C_0402_1005Metric, F.Cu at (634.3, 383.9)
- added C260: 1µF/25V, Capacitor_SMD:C_0805_2012Metric, F.Cu at (1160.8, 833.0)
- added C261: 1µF/6.3V, Capacitor_SMD:C_0603_1608Metric_Pad1.08x0.95mm_HandSolder, F.Cu at (1166.6, 796.2)
- added C262: 100nF, Capacitor_SMD:C_0805_2012Metric, F.Cu at (1169.7, 833.0)
- added C263: 1µF/6.3V, Capacitor_SMD:C_0603_1608Metric_Pad1.08x0.95mm_HandSolder, F.Cu at (1173.5, 796.2)
- added C264: 1µF/6.3V, Capacitor_SMD:C_0603_1608Metric_Pad1.08x0.95mm_HandSolder, F.Cu at (1179.9, 796.2)
- added C265: 1µF/6.3V, Capacitor_SMD:C_0603_1608Metric_Pad1.08x0.95mm_HandSolder, F.Cu at (1181.8, 827.9)
- added C266: 1µF/6.3V, Capacitor_SMD:C_0603_1608Metric_Pad1.08x0.95mm_HandSolder, F.Cu at (1185.0, 827.9)
- added C267: 1µF/6.3V, Capacitor_SMD:C_0603_1608Metric_Pad1.08x0.95mm_HandSolder, F.Cu at (1185.6, 796.2)
- added C268: 1µF/6.3V, Capacitor_SMD:C_0603_1608Metric_Pad1.08x0.95mm_HandSolder, F.Cu at (1231.5, 827.6)
- added C269: 1µF/6.3V, Capacitor_SMD:C_0603_1608Metric_Pad1.08x0.95mm_HandSolder, F.Cu at (1235.3, 827.6)
- added C27: 100nF, Capacitor_SMD:C_0402_1005Metric, F.Cu at (666.6, 331.2)
- added C270: 1µF/6.3V, Capacitor_SMD:C_0603_1608Metric_Pad1.08x0.95mm_HandSolder, F.Cu at (1235.9, 795.9)
- added C271: 1µF/6.3V, Capacitor_SMD:C_0603_1608Metric_Pad1.08x0.95mm_HandSolder, F.Cu at (1241.6, 795.9)
- added C272: 1µF/6.3V, Capacitor_SMD:C_0603_1608Metric_Pad1.08x0.95mm_HandSolder, F.Cu at (1247.3, 795.9)
- added C273: 10µF/25V, Capacitor_SMD:C_0805_2012Metric, F.Cu at (1251.8, 832.7)
- added C274: 1µF/6.3V, Capacitor_SMD:C_0603_1608Metric_Pad1.08x0.95mm_HandSolder, F.Cu at (1255.6, 795.9)
- added C275: 100µ/6.3V, Capacitor_SMD:C_1206_3216Metric, F.Cu at (1260.0, 782.6)
- added C276: 1µF/25V, Capacitor_SMD:C_0805_2012Metric, F.Cu at (1260.0, 832.7)
- added C277: 1µF/6.3V, Capacitor_SMD:C_0603_1608Metric_Pad1.08x0.95mm_HandSolder, F.Cu at (1265.8, 795.9)
- added C278: 100nF, Capacitor_SMD:C_0805_2012Metric, F.Cu at (1268.9, 832.7)
- added C279: 1µF/6.3V, Capacitor_SMD:C_0603_1608Metric_Pad1.08x0.95mm_HandSolder, F.Cu at (1272.7, 795.9)
- added C28: 470µ/25V, Capacitor_SMD:CP_Elec_8x10, F.Cu at (855.8, 454.4)
- added C280: 1µF/6.3V, Capacitor_SMD:C_0603_1608Metric_Pad1.08x0.95mm_HandSolder, F.Cu at (1279.1, 795.9)
- added C281: 1µF/6.3V, Capacitor_SMD:C_0603_1608Metric_Pad1.08x0.95mm_HandSolder, F.Cu at (1281.0, 827.6)
- added C282: 1µF/6.3V, Capacitor_SMD:C_0603_1608Metric_Pad1.08x0.95mm_HandSolder, F.Cu at (1284.2, 827.6)
- added C283: 1µF/6.3V, Capacitor_SMD:C_0603_1608Metric_Pad1.08x0.95mm_HandSolder, F.Cu at (1284.8, 795.9)
- added C284: 1µF/6.3V, Capacitor_SMD:C_0603_1608Metric_Pad1.08x0.95mm_HandSolder, F.Cu at (1337.3, 827.9)
- added C285: 1µF/6.3V, Capacitor_SMD:C_0603_1608Metric_Pad1.08x0.95mm_HandSolder, F.Cu at (1341.1, 827.9)
- added C286: 1µF/6.3V, Capacitor_SMD:C_0603_1608Metric_Pad1.08x0.95mm_HandSolder, F.Cu at (1341.7, 796.1)
- added C287: 1µF/6.3V, Capacitor_SMD:C_0603_1608Metric_Pad1.08x0.95mm_HandSolder, F.Cu at (1347.4, 796.1)
- added C288: 1µF/6.3V, Capacitor_SMD:C_0603_1608Metric_Pad1.08x0.95mm_HandSolder, F.Cu at (1353.1, 796.1)
- added C289: 10µF/25V, Capacitor_SMD:C_0805_2012Metric, F.Cu at (1357.6, 833.0)
- added C29: 470µ/25V, Capacitor_SMD:CP_Elec_8x10, F.Cu at (865.1, 454.7)
- added C290: 1µF/6.3V, Capacitor_SMD:C_0603_1608Metric_Pad1.08x0.95mm_HandSolder, F.Cu at (1361.4, 796.1)
- added C291: 100µ/6.3V, Capacitor_SMD:C_1206_3216Metric, F.Cu at (1365.8, 782.8)
- added C292: 1µF/25V, Capacitor_SMD:C_0805_2012Metric, F.Cu at (1365.8, 833.0)
- added C293: 1µF/6.3V, Capacitor_SMD:C_0603_1608Metric_Pad1.08x0.95mm_HandSolder, F.Cu at (1371.5, 796.1)
- added C294: 100nF, Capacitor_SMD:C_0805_2012Metric, F.Cu at (1374.7, 833.0)
- added C295: 1µF/6.3V, Capacitor_SMD:C_0603_1608Metric_Pad1.08x0.95mm_HandSolder, F.Cu at (1378.5, 796.1)
- added C296: 1µF/6.3V, Capacitor_SMD:C_0603_1608Metric_Pad1.08x0.95mm_HandSolder, F.Cu at (1384.9, 796.1)
- added C297: 1µF/6.3V, Capacitor_SMD:C_0603_1608Metric_Pad1.08x0.95mm_HandSolder, F.Cu at (1386.8, 827.9)
- added C298: 1µF/6.3V, Capacitor_SMD:C_0603_1608Metric_Pad1.08x0.95mm_HandSolder, F.Cu at (1390.0, 827.9)
- added C299: 1µF/6.3V, Capacitor_SMD:C_0603_1608Metric_Pad1.08x0.95mm_HandSolder, F.Cu at (1390.6, 796.1)
- added C3: 100nF, Capacitor_SMD:C_0402_1005Metric, F.Cu at (558.1, 373.8)
- added C30: 470µ/25V, Capacitor_SMD:CP_Elec_8x10, F.Cu at (874.3, 454.4)
- added C300: 1µF/6.3V, Capacitor_SMD:C_0603_1608Metric_Pad1.08x0.95mm_HandSolder, F.Cu at (1445.1, 830.6)
- added C301: 1µF/6.3V, Capacitor_SMD:C_0603_1608Metric_Pad1.08x0.95mm_HandSolder, F.Cu at (1448.9, 830.6)
- added C302: 1µF/6.3V, Capacitor_SMD:C_0603_1608Metric_Pad1.08x0.95mm_HandSolder, F.Cu at (1449.5, 798.9)
- added C303: 1µF/6.3V, Capacitor_SMD:C_0603_1608Metric_Pad1.08x0.95mm_HandSolder, F.Cu at (1455.2, 798.9)
- added C304: 1µF/6.3V, Capacitor_SMD:C_0603_1608Metric_Pad1.08x0.95mm_HandSolder, F.Cu at (1460.9, 798.9)
- added C305: 10µF/25V, Capacitor_SMD:C_0805_2012Metric, F.Cu at (1465.4, 835.7)
- added C306: 1µF/6.3V, Capacitor_SMD:C_0603_1608Metric_Pad1.08x0.95mm_HandSolder, F.Cu at (1469.2, 798.9)
- added C307: 100µ/6.3V, Capacitor_SMD:C_1206_3216Metric, F.Cu at (1473.6, 785.5)
- added C308: 1µF/25V, Capacitor_SMD:C_0805_2012Metric, F.Cu at (1473.6, 835.7)
- added C309: 1µF/6.3V, Capacitor_SMD:C_0603_1608Metric_Pad1.08x0.95mm_HandSolder, F.Cu at (1479.3, 798.9)
- added C31: 10µF/25V, Capacitor_SMD:C_0805_2012Metric, F.Cu at (865.4, 557.3)
- added C310: 100nF, Capacitor_SMD:C_0805_2012Metric, F.Cu at (1482.5, 835.7)
- added C311: 1µF/6.3V, Capacitor_SMD:C_0603_1608Metric_Pad1.08x0.95mm_HandSolder, F.Cu at (1486.3, 798.9)
- added C312: 1µF/6.3V, Capacitor_SMD:C_0603_1608Metric_Pad1.08x0.95mm_HandSolder, F.Cu at (1492.7, 798.9)
- added C313: 1µF/6.3V, Capacitor_SMD:C_0603_1608Metric_Pad1.08x0.95mm_HandSolder, F.Cu at (1494.6, 830.6)
- added C314: 1µF/6.3V, Capacitor_SMD:C_0603_1608Metric_Pad1.08x0.95mm_HandSolder, F.Cu at (1497.8, 830.6)
- added C315: 1µF/6.3V, Capacitor_SMD:C_0603_1608Metric_Pad1.08x0.95mm_HandSolder, F.Cu at (1498.4, 798.9)
- added C316: 1µF/6.3V, Capacitor_SMD:C_0603_1608Metric_Pad1.08x0.95mm_HandSolder, F.Cu at (1548.3, 829.6)
- added C317: 1µF/6.3V, Capacitor_SMD:C_0603_1608Metric_Pad1.08x0.95mm_HandSolder, F.Cu at (1552.1, 829.6)
- added C318: 1µF/6.3V, Capacitor_SMD:C_0603_1608Metric_Pad1.08x0.95mm_HandSolder, F.Cu at (1552.8, 797.8)
- added C319: 1µF/6.3V, Capacitor_SMD:C_0603_1608Metric_Pad1.08x0.95mm_HandSolder, F.Cu at (1558.5, 797.8)
- added C32: 22pF, Capacitor_SMD:C_0805_2012Metric, F.Cu at (866.6, 522.7)
- added C320: 1µF/6.3V, Capacitor_SMD:C_0603_1608Metric_Pad1.08x0.95mm_HandSolder, F.Cu at (1564.2, 797.8)
- added C321: 10µF/25V, Capacitor_SMD:C_0805_2012Metric, F.Cu at (1568.6, 834.6)
- added C322: 1µF/6.3V, Capacitor_SMD:C_0603_1608Metric_Pad1.08x0.95mm_HandSolder, F.Cu at (1572.4, 797.8)
- added C323: 100µ/6.3V, Capacitor_SMD:C_1206_3216Metric, F.Cu at (1576.9, 784.5)
- added C324: 1µF/25V, Capacitor_SMD:C_0805_2012Metric, F.Cu at (1576.9, 834.6)
- added C325: 1µF/6.3V, Capacitor_SMD:C_0603_1608Metric_Pad1.08x0.95mm_HandSolder, F.Cu at (1582.6, 797.8)
- added C326: 100nF, Capacitor_SMD:C_0805_2012Metric, F.Cu at (1585.8, 834.6)
- added C327: 1µF/6.3V, Capacitor_SMD:C_0603_1608Metric_Pad1.08x0.95mm_HandSolder, F.Cu at (1589.6, 797.8)
- added C328: 1µF/6.3V, Capacitor_SMD:C_0603_1608Metric_Pad1.08x0.95mm_HandSolder, F.Cu at (1595.9, 797.8)
- added C329: 1µF/6.3V, Capacitor_SMD:C_0603_1608Metric_Pad1.08x0.95mm_HandSolder, F.Cu at (1597.8, 829.6)
- added C33: 100pF, Capacitor_SMD:C_0805_2012Metric, F.Cu at (866.6, 525.2)
- added C330: 1µF/6.3V, Capacitor_SMD:C_0603_1608Metric_Pad1.08x0.95mm_HandSolder, F.Cu at (1601.0, 829.6)
- added C331: 1µF/6.3V, Capacitor_SMD:C_0603_1608Metric_Pad1.08x0.95mm_HandSolder, F.Cu at (1601.7, 797.8)
- added C332: 1µF/6.3V, Capacitor_SMD:C_0603_1608Metric_Pad1.08x0.95mm_HandSolder, F.Cu at (1644.9, 827.5)
- added C333: 1µF/6.3V, Capacitor_SMD:C_0603_1608Metric_Pad1.08x0.95mm_HandSolder, F.Cu at (1648.7, 827.5)
- added C334: 1µF/6.3V, Capacitor_SMD:C_0603_1608Metric_Pad1.08x0.95mm_HandSolder, F.Cu at (1649.4, 795.7)
- added C335: 1µF/6.3V, Capacitor_SMD:C_0603_1608Metric_Pad1.08x0.95mm_HandSolder, F.Cu at (1655.1, 795.7)
- added C336: 1µF/6.3V, Capacitor_SMD:C_0603_1608Metric_Pad1.08x0.95mm_HandSolder, F.Cu at (1660.8, 795.7)
- added C337: 10µF/25V, Capacitor_SMD:C_0805_2012Metric, F.Cu at (1665.2, 832.6)
- added C338: 1µF/6.3V, Capacitor_SMD:C_0603_1608Metric_Pad1.08x0.95mm_HandSolder, F.Cu at (1669.0, 795.7)
- added C339: 100µ/6.3V, Capacitor_SMD:C_1206_3216Metric, F.Cu at (1673.5, 782.4)
- added C34: 22pF, Capacitor_SMD:C_0805_2012Metric, F.Cu at (866.6, 527.8)
- added C340: 1µF/25V, Capacitor_SMD:C_0805_2012Metric, F.Cu at (1673.5, 832.6)
- added C341: 1µF/6.3V, Capacitor_SMD:C_0603_1608Metric_Pad1.08x0.95mm_HandSolder, F.Cu at (1679.2, 795.7)
- added C342: 100nF, Capacitor_SMD:C_0805_2012Metric, F.Cu at (1682.4, 832.6)
- added C343: 1µF/6.3V, Capacitor_SMD:C_0603_1608Metric_Pad1.08x0.95mm_HandSolder, F.Cu at (1686.2, 795.7)
- added C344: 1µF/6.3V, Capacitor_SMD:C_0603_1608Metric_Pad1.08x0.95mm_HandSolder, F.Cu at (1692.5, 795.7)
- added C345: 1µF/6.3V, Capacitor_SMD:C_0603_1608Metric_Pad1.08x0.95mm_HandSolder, F.Cu at (1694.5, 827.5)
- added C346: 1µF/6.3V, Capacitor_SMD:C_0603_1608Metric_Pad1.08x0.95mm_HandSolder, F.Cu at (1697.6, 827.5)
- added C347: 1µF/6.3V, Capacitor_SMD:C_0603_1608Metric_Pad1.08x0.95mm_HandSolder, F.Cu at (1698.3, 795.7)
- added C348: 1µF/6.3V, Capacitor_SMD:C_0603_1608Metric_Pad1.08x0.95mm_HandSolder, F.Cu at (1746.5, 829.5)
- added C349: 1µF/6.3V, Capacitor_SMD:C_0603_1608Metric_Pad1.08x0.95mm_HandSolder, F.Cu at (1750.3, 829.5)
- added C35: 470µ/25V, Capacitor_SMD:CP_Elec_8x10, F.Cu at (883.5, 454.4)
- added C350: 1µF/6.3V, Capacitor_SMD:C_0603_1608Metric_Pad1.08x0.95mm_HandSolder, F.Cu at (1750.9, 797.7)
- added C351: 1µF/6.3V, Capacitor_SMD:C_0603_1608Metric_Pad1.08x0.95mm_HandSolder, F.Cu at (1756.6, 797.7)
- added C352: 1µF/6.3V, Capacitor_SMD:C_0603_1608Metric_Pad1.08x0.95mm_HandSolder, F.Cu at (1762.3, 797.7)
- added C353: 10µF/25V, Capacitor_SMD:C_0805_2012Metric, F.Cu at (1766.8, 834.6)
- added C354: 1µF/6.3V, Capacitor_SMD:C_0603_1608Metric_Pad1.08x0.95mm_HandSolder, F.Cu at (1770.6, 797.7)
- added C355: 100µ/6.3V, Capacitor_SMD:C_1206_3216Metric, F.Cu at (1775.0, 784.4)
- added C356: 1µF/25V, Capacitor_SMD:C_0805_2012Metric, F.Cu at (1775.0, 834.6)
- added C357: 1µF/6.3V, Capacitor_SMD:C_0603_1608Metric_Pad1.08x0.95mm_HandSolder, F.Cu at (1780.8, 797.7)
- added C358: 100nF, Capacitor_SMD:C_0805_2012Metric, F.Cu at (1783.9, 834.6)
- added C359: 1µF/6.3V, Capacitor_SMD:C_0603_1608Metric_Pad1.08x0.95mm_HandSolder, F.Cu at (1787.7, 797.7)
- added C36: 1nF, Capacitor_SMD:C_0805_2012Metric, F.Cu at (869.5, 511.9)
- added C360: 1µF/6.3V, Capacitor_SMD:C_0603_1608Metric_Pad1.08x0.95mm_HandSolder, F.Cu at (1794.1, 797.7)
- added C361: 1µF/6.3V, Capacitor_SMD:C_0603_1608Metric_Pad1.08x0.95mm_HandSolder, F.Cu at (1796.0, 829.5)
- added C362: 1µF/6.3V, Capacitor_SMD:C_0603_1608Metric_Pad1.08x0.95mm_HandSolder, F.Cu at (1799.2, 829.5)
- added C363: 1µF/6.3V, Capacitor_SMD:C_0603_1608Metric_Pad1.08x0.95mm_HandSolder, F.Cu at (1799.8, 797.7)
- added C364: 0.1uF, Capacitor_SMD:C_0805_2012Metric, F.Cu at (1159.1, 219.8)
- added C365: 27pf, Capacitor_SMD:C_0805_2012Metric, F.Cu at (1189.6, 387.2)
- added C366: 4.7uF, Capacitor_SMD:C_0805_2012Metric, F.Cu at (1194.7, 326.8)
- added C367: 4.7uF, Capacitor_SMD:C_0805_2012Metric, F.Cu at (1201.7, 326.8)
- added C368: 27pf, Capacitor_SMD:C_0805_2012Metric, F.Cu at (1203.6, 387.2)
- added C369: 0.1uF, Capacitor_SMD:C_0805_2012Metric, F.Cu at (1208.0, 326.8)
- added C37: 1nF, Capacitor_SMD:C_0805_2012Metric, F.Cu at (871.4, 478.2)
- added C370: 3.3uF, Capacitor_SMD:C_0805_2012Metric, F.Cu at (1209.9, 353.5)
- added C371: 0.1uF, Capacitor_SMD:C_0805_2012Metric, F.Cu at (1215.0, 326.8)
- added C372: 0.1uF, Capacitor_SMD:C_0805_2012Metric, F.Cu at (1260.7, 342.7)
- added C373: 0.1uF, Capacitor_SMD:C_0805_2012Metric, F.Cu at (1267.7, 342.7)
- added C374: 0.1uF, Capacitor_SMD:C_0805_2012Metric, F.Cu at (1274.1, 342.7)
- added C375: 0.1uF, Capacitor_SMD:C_0805_2012Metric, F.Cu at (1280.4, 342.7)
- added C376: 0.1uF, Capacitor_SMD:C_0805_2012Metric, F.Cu at (1286.8, 342.7)
- added C377: 0.1uF, Capacitor_SMD:C_0805_2012Metric, F.Cu at (1293.1, 342.7)
- added C378: 0.1uF, Capacitor_SMD:C_0805_2012Metric, F.Cu at (1299.5, 342.7)
- added C38: 22µ/25V, Capacitor_SMD:C_1210_3225Metric, F.Cu at (889.5, 454.4)
- added C39: 22µ/25V, Capacitor_SMD:C_1210_3225Metric, F.Cu at (892.5, 454.4)
- added C4: 100nF, Capacitor_SMD:C_0402_1005Metric, F.Cu at (558.1, 390.3)
- added C40: 10nF, Capacitor_SMD:C_0805_2012Metric, F.Cu at (881.2, 551.6)
- added C41: 22µ/25V, Capacitor_SMD:C_1210_3225Metric, F.Cu at (895.5, 454.4)
- added C42: 22µ/25V, Capacitor_SMD:C_1210_3225Metric, F.Cu at (898.6, 454.4)
- added C43: 22µ/25V, Capacitor_SMD:C_1210_3225Metric, F.Cu at (901.6, 454.4)
- added C44: 22µ/25V, Capacitor_SMD:C_1210_3225Metric, F.Cu at (893.9, 558.6)
- added C45: 22µ/25V, Capacitor_SMD:C_1210_3225Metric, F.Cu at (904.6, 454.4)
- added C46: 22µ/25V, Capacitor_SMD:C_1210_3225Metric, F.Cu at (907.7, 454.4)
- added C47: 22µ/25V, Capacitor_SMD:C_1210_3225Metric, F.Cu at (910.7, 454.4)
- added C48: 22µ/25V, Capacitor_SMD:C_1210_3225Metric, F.Cu at (913.7, 454.4)
- added C49: 22µ/25V, Capacitor_SMD:C_1210_3225Metric, F.Cu at (916.8, 454.4)
- added C5: 100nF, Capacitor_SMD:C_0402_1005Metric, F.Cu at (560.6, 373.8)
- added C50: 4.7µF/16V, Capacitor_SMD:C_0805_2012Metric, F.Cu at (917.1, 483.9)
- added C51: 1µF/25V, Capacitor_SMD:C_0805_2012Metric, F.Cu at (917.1, 491.6)
- added C52: 22µ/25V, Capacitor_SMD:C_1210_3225Metric, F.Cu at (919.8, 454.4)
- added C53: 1µF/25V, Capacitor_SMD:C_0805_2012Metric, F.Cu at (920.9, 483.9)
- added C54: 22µ/25V, Capacitor_SMD:C_1210_3225Metric, F.Cu at (922.8, 454.4)
- added C55: 330nF, Capacitor_SMD:C_0805_2012Metric, F.Cu at (923.5, 491.6)
- added C56: 12pF, Capacitor_SMD:C_0805_2012Metric, F.Cu at (925.4, 503.0)
- added C57: 2.2nF, Capacitor_SMD:C_0805_2012Metric, F.Cu at (927.3, 511.3)
- added C58: 1nF, Capacitor_SMD:C_0805_2012Metric, F.Cu at (928.5, 499.8)
- added C59: 330µF/4V, Capacitor_SMD:C_1210_3225Metric, F.Cu at (972.7, 472.8)
- added C6: 100nF, Capacitor_SMD:C_0402_1005Metric, F.Cu at (560.6, 390.3)
- added C60: 100µ/6.3V, Capacitor_SMD:C_1206_3216Metric, F.Cu at (973.3, 492.5)
- added C61: 100µ/6.3V, Capacitor_SMD:C_1206_3216Metric, F.Cu at (973.3, 512.8)
- added C62: 330µF/4V, Capacitor_SMD:C_1210_3225Metric, F.Cu at (975.2, 472.8)
- added C63: 100µ/6.3V, Capacitor_SMD:C_1206_3216Metric, F.Cu at (976.5, 492.5)
- added C64: 100µ/6.3V, Capacitor_SMD:C_1206_3216Metric, F.Cu at (976.5, 512.8)
- added C65: 330µF/4V, Capacitor_SMD:C_1210_3225Metric, F.Cu at (977.8, 472.8)
- added C66: 330µF/4V, Capacitor_SMD:C_1210_3225Metric, F.Cu at (980.3, 472.8)
- added C67: 100µ/6.3V, Capacitor_SMD:C_1206_3216Metric, F.Cu at (980.3, 492.5)
- added C68: 100µ/6.3V, Capacitor_SMD:C_1206_3216Metric, F.Cu at (980.3, 512.8)
- added C69: 330µF/4V, Capacitor_SMD:C_1210_3225Metric, F.Cu at (982.8, 472.8)
- added C7: 100nF, Capacitor_SMD:C_0402_1005Metric, F.Cu at (563.1, 373.8)
- added C70: 100µ/6.3V, Capacitor_SMD:C_1206_3216Metric, F.Cu at (983.5, 492.5)
- added C71: 100µ/6.3V, Capacitor_SMD:C_1206_3216Metric, F.Cu at (983.5, 512.8)
- added C72: 330µF/4V, Capacitor_SMD:C_1210_3225Metric, F.Cu at (983.5, 540.1)
- added C73: 330µF/4V, Capacitor_SMD:C_1210_3225Metric, F.Cu at (985.4, 472.8)
- added C74: 100µ/6.3V, Capacitor_SMD:C_1206_3216Metric, F.Cu at (986.6, 492.5)
- added C75: 100µ/6.3V, Capacitor_SMD:C_1206_3216Metric, F.Cu at (986.6, 512.8)
- added C76: 330µF/4V, Capacitor_SMD:C_1210_3225Metric, F.Cu at (987.9, 472.8)
- added C77: 330µF/4V, Capacitor_SMD:C_1210_3225Metric, F.Cu at (988.6, 540.1)
- added C78: 100µ/6.3V, Capacitor_SMD:C_1206_3216Metric, F.Cu at (989.8, 492.5)
- added C79: 100µ/6.3V, Capacitor_SMD:C_1206_3216Metric, F.Cu at (989.8, 512.8)
- added C8: 100nF, Capacitor_SMD:C_0402_1005Metric, F.Cu at (563.1, 390.3)
- added C80: 330µF/4V, Capacitor_SMD:C_1210_3225Metric, F.Cu at (990.5, 472.8)
- added C81: 330µF/4V, Capacitor_SMD:C_1210_3225Metric, F.Cu at (993.0, 472.8)
- added C82: 100µ/6.3V, Capacitor_SMD:C_1206_3216Metric, F.Cu at (993.0, 492.5)
- added C83: 100µ/6.3V, Capacitor_SMD:C_1206_3216Metric, F.Cu at (993.0, 512.8)
- added C84: 330µF/4V, Capacitor_SMD:C_1210_3225Metric, F.Cu at (993.6, 540.1)
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Connections:
- net /~{PRSNT2x4} renamed /PCIexpress_connector/~{PRSNT2x4}
- J2 pad B10: +3.3VA -> unconnected-(J2-+3.3V_aux-PadB10)
Other:
- outline, holes or cut-outs redrawn
