File: PC-AXE.kicad_pcb (KiCad board)
At the start: 6 copper layers, 312 x 111.2 mm, 565 parts, among them J1 PCIexpress_bracket, J10 61900411021, J2 PCIexpress_x4, J3 353180620, J4 353180620, J5 353180620, J6 Conn_01x06, J7 61900411021, J8 61900411021, J9 61900411021, U1 TLV62568ADRLR, U10 CSD95472Q5MC, U11 CSD95472Q5MC, U12 CSD95472Q5MC, U13 25MHz, U14 TXU0304PW, U15 MCP1824T-0802E, U16 MCP1824T-1202E, U17 BM1370_mode1, U18 BM1370_mode1, U19 BM1370_mode1, U2 AP2204K-1.8, U20 BM1370_mode1, U21 BM1370_mode1, U22 BM1370_mode1, U23 BM1370_mode1, U24 BM1370_mode1, U25 BM1370_mode1, U26 BM1370_mode1, U27 BM1370_mode1, U28 BM1370_mode1, U29 EMC2305, U3 VL805, U30 M93C46-WDW6TP, U31 FT4232HQ, U4 W25Q32JVZP, U5 AP3211, U6 TPS53667RTAR, U7 CSD95472Q5MC, U8 CSD95472Q5MC, U9 CSD95472Q5MC, Y1 25Mhz, Y2 12MHz

Commit message: Updated after DRC
Parts:
- moved C151 0.25 mm to (238.3, 170.8)
- moved C182 0.11 mm to (280.3, 120.7)
- moved C14 0.10 mm to (142.0, 168.7)
- moved C294 0.08 mm to (286.6, 145.6)
- moved C196 0.07 mm to (306.9, 120.7)
Connections:
- U31 pad 24: unconnected-(U31-ADBUS7-Pad24) -> /LDO_EN
Routing:
- net +12V: track 4.91 -> 2.28 mm
- net +3V3: track 718.7 -> 719.4 mm
- net GND: vias 1580 -> 1574
