File: bm1370.kicad_sch (KiCad schematic)
At the start: 20 parts, among them U17 BM1370_mode1

Commit message: updated schematic working on layout
Other:
- company: (none) -> Author: Aadhi M
- title: (none) -> PC-AXE
Changed lines of the file:
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@@
 	(generator_version "9.0")
 	(paper "A4")
+	(title_block
+		(title "PC-AXE")
+		(company "Author: Aadhi M")
+	)
 	(junction
 		(at 121.92 106.68)
