File: power_stage.kicad_sch (KiCad schematic)
At the start: 12 parts, among them U7 CSD95472Q5MC

Commit message: updated schematic working on layout
Parts:
- renumbered C109 to C127, C110 to C128, C111 to C129, C112 to C130, C113 to C131, C114 to C132, C115 to C133, C116 to C134, L3 to L5, R32 to R38, R33 to R39, U7 to U9
Other:
- company: (none) -> Author: Aadhi M
- title: (none) -> PC-AXE
Changed lines of the file:
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@@
 	(generator_version "9.0")
 	(paper "A4")
+	(title_block
+		(title "PC-AXE")
+		(company "Author: Aadhi M")
+	)
 	(junction
 		(at 92.71 64.77)
@@
 		(dnp no)
 		(fields_autoplaced yes)
-		(property "Reference" "#PWR0120"
+		(property "Reference" "#PWR0142"
 			(at 109.22 59.69 0)
 			(effects
@@
 		(on_board yes)
 		(dnp no)
-		(property "Reference" "C111"
+		(property "Reference" "C129"
 			(at 115.57 52.07 0)
 			(effects
@@
 		(on_board yes)
 		(dnp no)
-		(property "Reference" "C115"
+		(property "Reference" "C133"
 			(at 169.672 91.694 0)
 			(effects
@@
 		(dnp no)
 		(fields_autoplaced yes)
-		(property "Reference" "#PWR0124"
+		(property "Reference" "#PWR0146"
 			(at 135.89 132.08 0)
 			(effects
@@
 		(on_board yes)
 		(dnp no)
-		(property "Reference" "L3"
+		(property "Reference" "L5"
 			(at 202.565 102.235 90)
 			(effects
@@
 		(dnp no)
 		(fields_autoplaced yes)
-		(property "Reference" "#PWR0119"
+		(property "Reference" "#PWR0141"
 			(at 101.6 83.82 0)
 			(effects
@@
 		(dnp no)
 		(fields_autoplaced yes)
-		(property "Reference" "#PWR0123"
+		(property "Reference" "#PWR0145"
 			(at 123.19 100.33 0)
 			(effects
@@
 		(on_board yes)
 		(dnp no)
-		(property "Reference" "C110"
+		(property "Reference" "C128"
 			(at 100.33 71.12 90)
 			(effects
@@
 		(on_board yes)
 		(dnp no)
-		(property "Reference" "R32"
+		(property "Reference" "R38"
 			(at 127 100.33 90)
 			(effects
@@
 		(on_board yes)
 		(dnp no)
-		(property "Reference" "#REF01"
+		(property "Reference" "#REF03"
 			(at 121.92 107.95 0)
 			(effects
@@
 		(on_board yes)
 		(dnp no)
-		(property "Reference" "#PWR0118"
+		(property "Reference" "#PWR0140"
 			(at 92.71 83.82 0)
 			(effects
@@
 		(dnp no)
 		(fields_autoplaced yes)
-		(property "Reference" "U7"
+		(property "Reference" "U9"
 			(at 152.4 82.55 0)
 			(effects
@@
 		(on_board yes)
 		(dnp no)
-		(property "Reference" "#PWR0117"
+		(property "Reference" "#PWR0139"
 			(at 83.82 64.77 0)
 			(effects
@@
 		(on_board yes)
 		(dnp no)
-		(property "Reference" "R33"
+		(property "Reference" "R39"
 			(at 185.42 116.84 90)
 			(effects
@@
 		(dnp no)
 		(fields_autoplaced yes)
-		(property "Reference" "C114"
+		(property "Reference" "C132"
 			(at 139.7 120.6499 0)
 			(effects
@@
 		(dnp no)
 		(fields_autoplaced yes)
-		(property "Reference" "#PWR0126"
+		(property "Reference" "#PWR0148"
 			(at 182.88 133.35 0)
 			(effects
@@
 		(on_board yes)
 		(dnp no)
-		(property "Reference" "C113"
+		(property "Reference" "C131"
 			(at 114.3 120.6499 0)
 			(effects
@@
 		(on_board yes)
 		(dnp no)
-		(property "Reference" "C116"
+		(property "Reference" "C134"
 			(at 191.516 122.936 0)
 			(effects
@@
 		(dnp no)
 		(fields_autoplaced yes)
-		(property "Reference" "#PWR0125"
+		(property "Reference" "#PWR0147"
 			(at 167.64 119.38 0)
 			(effects
@@
 		(on_board yes)
 		(dnp no)
-		(property "Reference" "C112"
+		(property "Reference" "C130"
 			(at 109.22 71.12 90)
 			(effects
@@
 		(dnp no)
 		(fields_autoplaced yes)
-		(property "Reference" "#PWR0122"
+		(property "Reference" "#PWR0144"
 			(at 118.11 132.08 0)
 			(effects
@@
 		(on_board yes)
 		(dnp no)
-		(property "Reference" "C109"
+		(property "Reference" "C127"
 			(at 91.44 71.12 90)
 			(effects
@@
 		(dnp no)
 		(fields_autoplaced yes)
-		(property "Reference" "#PWR0121"
+		(property "Reference" "#PWR0143"
 			(at 110.49 83.82 0)
 			(effects
