File: term.kicad_sch (KiCad schematic)
At the start: 2 parts

Commit message: updated schematic working on layout
Other:
- company: Author: Luca Anastasio -> Author: Aadhi M
- title: PCIexpress_x4_full -> PC-AXE
Changed lines of the file:
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@@
 	(paper "A4")
 	(title_block
-		(title "PCIexpress_x4_full")
-		(company "Author: Luca Anastasio")
+		(title "PC-AXE")
+		(company "Author: Aadhi M")
 	)
 	(junction
