File: untitled.kicad_sch (KiCad schematic)
At the start: 43 parts, among them U1 TLV62568ADRLR, U2 AP2204K-1.8, U3 VL805, U4 W25Q32JVZP, Y1 25Mhz

Commit message: board stakup updated and schematic is updated
Connections:
- no-connect marks 0 -> 23
Changed lines of the file:
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@@
+	)
+	(junction
+		(at 114.3 44.45)
+		(diameter 0)
+		(color 0 0 0 0)
 	)
 	(junction
@@
 	(junction
 		(at 62.23 165.1)
-		(diameter 0)
-		(color 0 0 0 0)
-	)
-	(junction
-		(at 114.3 44.45)
 		(diameter 0)
 		(color 0 0 0 0)
@@
 		(color 0 0 0 0)
 	)
+	(no_connect
+		(at 172.72 73.66)
+	)
+	(no_connect
+		(at 172.72 49.53)
+	)
+	(no_connect
+		(at 172.72 71.12)
+	)
+	(no_connect
+		(at 172.72 41.91)
+	)
+	(no_connect
+		(at 172.72 114.3)
+	)
+	(no_connect
+		(at 172.72 83.82)
+	)
+	(no_connect
+		(at 172.72 102.87)
+	)
+	(no_connect
+		(at 172.72 76.2)
+	)
+	(no_connect
+		(at 172.72 88.9)
+	)
+	(no_connect
+		(at 172.72 44.45)
+	)
+	(no_connect
+		(at 172.72 78.74)
+	)
+	(no_connect
+		(at 172.72 100.33)
+	)
+	(no_connect
+		(at 172.72 106.68)
+	)
+	(no_connect
+		(at 172.72 52.07)
+	)
+	(no_connect
+		(at 172.72 109.22)
+	)
+	(no_connect
+		(at 172.72 86.36)
+	)
+	(no_connect
+		(at 172.72 46.99)
+	)
+	(no_connect
+		(at 172.72 91.44)
+	)
+	(no_connect
+		(at 172.72 97.79)
+	)
+	(no_connect
+		(at 31.75 41.91)
+	)
+	(no_connect
+		(at 172.72 95.25)
+	)
+	(no_connect
+		(at 172.72 54.61)
+	)
+	(no_connect
+		(at 172.72 111.76)
+	)
 	(wire
 		(pts
@@
 	(wire
 		(pts
+			(xy 114.3 44.45) (xy 128.27 44.45)
+		)
+		(stroke
+			(width 0)
+			(type default)
+		)
+	)
+	(wire
+		(pts
 			(xy 111.76 81.28) (xy 115.57 81.28)
 		)
@@
 	(wire
 		(pts
-			(xy 114.3 44.45) (xy 128.27 44.45)
-		)
-		(stroke
-			(width 0)
-			(type default)
-		)
-	)
-	(wire
-		(pts
 			(xy 72.39 152.4) (xy 72.39 154.94)
 		)
@@
 	(wire
 		(pts
+			(xy 114.3 44.45) (xy 114.3 46.99)
+		)
+		(stroke
+			(width 0)
+			(type default)
+		)
+	)
+	(wire
+		(pts
 			(xy 118.11 86.36) (xy 128.27 86.36)
 		)
@@
 	(wire
 		(pts
+			(xy 57.15 162.56) (xy 57.15 165.1)
+		)
+		(stroke
+			(width 0)
+			(type default)
+		)
+	)
+	(wire
+		(pts
+			(xy 80.01 26.67) (xy 83.82 26.67)
+		)
+		(stroke
+			(width 0)
+			(type default)
+		)
+	)
+	(wire
+		(pts
+			(xy 41.91 132.08) (xy 46.99 132.08)
+		)
+		(stroke
+			(width 0)
+			(type default)
+		)
+	)
+	(wire
+		(pts
+			(xy 119.38 24.13) (xy 128.27 24.13)
+		)
+		(stroke
+			(width 0)
+			(type default)
+		)
+	)
+	(wire
+		(pts
+			(xy 232.41 36.83) (xy 226.06 36.83)
+		)
+		(stroke
+			(width 0)
+			(type default)
+		)
+	)
+	(wire
+		(pts
+			(xy 36.83 165.1) (xy 41.91 165.1)
+		)
+		(stroke
+			(width 0)
+			(type default)
+		)
+	)
+	(wire
+		(pts
+			(xy 172.72 130.81) (xy 181.61 130.81)
+		)
+		(stroke
+			(width 0)
+			(type default)
+		)
+	)
+	(wire
+		(pts
+			(xy 118.11 69.85) (xy 120.65 69.85)
+		)
+		(stroke
+			(width 0)
+			(type default)
+		)
+	)
+	(wire
+		(pts
+			(xy 111.76 64.77) (xy 128.27 64.77)
+		)
+		(stroke
+			(width 0)
+			(type default)
+		)
+	)
+	(wire
+		(pts
+			(xy 54.61 132.08) (xy 57.15 132.08)
+		)
+		(stroke
+			(width 0)
+			(type default)
+		)
+	)
+	(wire
+		(pts
 			(xy 114.3 41.91) (xy 114.3 44.45)
 		)
 		(stroke
-			(width 0)
-			(type default)
-		)
-	)
-	(wire
-		(pts
-			(xy 57.15 162.56) (xy 57.15 165.1)
-		)
-		(stroke
-			(width 0)
-			(type default)
-		)
-	)
-	(wire
-		(pts
-			(xy 80.01 26.67) (xy 83.82 26.67)
-		)
-		(stroke
-			(width 0)
-			(type default)
-		)
-	)
-	(wire
-		(pts
-			(xy 41.91 132.08) (xy 46.99 132.08)
-		)
-		(stroke
-			(width 0)
-			(type default)
-		)
-	)
-	(wire
-		(pts
-			(xy 119.38 24.13) (xy 128.27 24.13)
-		)
-		(stroke
-			(width 0)
-			(type default)
-		)
-	)
-	(wire
-		(pts
-			(xy 232.41 36.83) (xy 226.06 36.83)
-		)
-		(stroke
-			(width 0)
-			(type default)
-		)
-	)
-	(wire
-		(pts
-			(xy 36.83 165.1) (xy 41.91 165.1)
-		)
-		(stroke
-			(width 0)
-			(type default)
-		)
-	)
-	(wire
-		(pts
-			(xy 172.72 130.81) (xy 181.61 130.81)
-		)
-		(stroke
-			(width 0)
-			(type default)
-		)
-	)
-	(wire
-		(pts
-			(xy 118.11 69.85) (xy 120.65 69.85)
-		)
-		(stroke
-			(width 0)
-			(type default)
-		)
-	)
-	(wire
-		(pts
-			(xy 111.76 64.77) (xy 128.27 64.77)
-		)
-		(stroke
-			(width 0)
-			(type default)
-		)
-	)
-	(wire
-		(pts
-			(xy 54.61 132.08) (xy 57.15 132.08)
-		)
-		(stroke
-			(width 0)
-			(type default)
-		)
-	)
-	(wire
-		(pts
-			(xy 114.3 44.45) (xy 114.3 46.99)
-		)
-		(stroke

Commit message: updated schematic working on layout
Other:
- company: (none) -> Author: Aadhi M
- title: (none) -> PC-AXE
Changed lines of the file:
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@@
 	(generator_version "9.0")
 	(paper "A4")
+	(title_block
+		(title "PC-AXE")
+		(company "Author: Aadhi M")
+	)
 	(junction
 		(at 184.15 121.92)
