File: PC-AXE_backup_altium.kicad_pcb (KiCad board)
At the start: 6 copper layers, 312 x 111.2 mm, 565 parts, among them J1 PCIexpress_bracket, J10 61900411021, J2 PCIexpress_x4, J3 353180620, J4 353180620, J5 353180620, J6 Conn_01x06, J7 61900411021, J8 61900411021, J9 61900411021, U1 TLV62568ADRLR, U10 CSD95472Q5MC, U11 CSD95472Q5MC, U12 CSD95472Q5MC, U13 25MHz, U14 TXU0304PW, U15 MCP1824T-0802E, U16 MCP1824T-1202E, U17 BM1370_mode1, U18 BM1370_mode1, U19 BM1370_mode1, U2 AP2204K-1.8, U20 BM1370_mode1, U21 BM1370_mode1, U22 BM1370_mode1, U23 BM1370_mode1, U24 BM1370_mode1, U25 BM1370_mode1, U26 BM1370_mode1, U27 BM1370_mode1, U28 BM1370_mode1, U29 EMC2305, U3 VL805, U30 M93C46-WDW6TP, U31 FT4232HQ, U4 W25Q32JVZP, U5 AP3211, U6 TPS53667RTAR, U7 CSD95472Q5MC, U8 CSD95472Q5MC, U9 CSD95472Q5MC, Y1 25Mhz, Y2 12MHz

Commit message: Updated new layout and routing of PCB
Parts:
- moved C229 67.4 mm to (276.5, 73.1)
- moved C232 67.4 mm to (281.8, 75.3)
- moved C235 67.4 mm to (281.8, 77.1)
- moved C238 67.4 mm to (281.8, 103.2)
- moved C239 67.4 mm to (281.8, 104.9)
- moved C242 67.4 mm to (276.5, 107.2)
- moved C357 67.4 mm to (276.5, 116.9)
- moved C360 67.4 mm to (281.8, 119.3)
- moved C363 67.4 mm to (281.8, 120.9)
- moved R82 67.4 mm to (266.7, 126.4)
- moved TP10 67.4 mm to (259.6, 100.9)
- moved C142 67.4 mm to (151.8, 109.0)
- moved C152 67.4 mm to (151.8, 124.2)
- moved C153 67.4 mm to (141.8, 122.2)
- moved C154 67.4 mm to (151.1, 116.2)
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Routing:
- net GND: track 485.7 -> 469.0 mm
- net Net-(U31-REF): track 11.4 -> 12.0 mm
Other:
- board size 312 x 111.2 mm -> 312 x 111.1 mm
