File: PC-AXE.kicad_sch (KiCad schematic)
At the start: 0 parts

Commit message: Updated after DRC
Other:
- sheet USB_to_UART ports: added LDO_EN; removed none
Changed lines of the file:
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@@
+		)
+	)
+	(label "LDO_EN"
+		(at 166.37 33.02 180)
+		(effects
+			(font
+				(size 1.27 1.27)
+			)
+			(justify right bottom)
 		)
 	)
@@
 			(effects
 				(font
+					(size 1.27 1.27)
+				)
+				(justify left)
+			)
+		)
+		(pin "LDO_EN" output
+			(at 166.37 33.02 180)
+			(effects
+				(font
